File: pcb/ESP012-16-Channel-PWM1.sch (EAGLE design)
At the start: 27 parts, among them IC2 UA78M33DCY, J1 DCJ0202, Q1 IRLML2244TRPBF, Q2 IRLML2244TRPBF, Q3 IRLML2244TRPBF, Q4 IRLML2244TRPBF, Q5 IRLML2244TRPBF, Q6 IRLML2244TRPBF, Q7 IRLML2244TRPBF, Q8 IRLML2244TRPBF

Commit message: changed 12V supply for LEDs to thicker wire
Parts:
- added JP4: (no value), pinhead:PINHD-1X2
Connections:
- net VCC12: now also JP4.1, JP4.2
Changed lines of the file:
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@@
 <part name="GND12" library="supply1" deviceset="GND" device=""/>
 <part name="R1" library="rcl" deviceset="R-EU_" device="MELF0207R" value="100"/>
+<part name="JP4" library="pinhead" deviceset="PINHD-1X2" device=""/>
 </parts>
 <sheets>
@@
 <instance part="GND12" gate="1" x="43.18" y="27.94"/>
 <instance part="R1" gate="G$1" x="43.18" y="43.18" rot="R90"/>
+<instance part="JP4" gate="G$1" x="307.34" y="50.8"/>
 </instances>
 <busses>
@@
 <junction x="-10.16" y="83.82"/>
 </segment>
+<segment>
+<pinref part="JP4" gate="G$1" pin="1"/>
+<wire x1="304.8" y1="53.34" x2="287.02" y2="53.34" width="0.1524" layer="91"/>
+<label x="287.02" y="53.34" size="1.778" layer="95"/>
+</segment>
+<segment>
+<pinref part="JP4" gate="G$1" pin="2"/>
+<wire x1="304.8" y1="50.8" x2="287.02" y2="50.8" width="0.1524" layer="91"/>
+<label x="287.02" y="50.8" size="1.778" layer="95"/>
+</segment>
 </net>
